File: pcb-bldc-servo-2/pcb-bldc-servo-2.brd (EAGLE design)
At the start: 36.5 x 29 mm, 38 parts, among them J1 03-JST-B3B-XH-A, U1 STM32G030F6P6, U2 DRV8870TH, U3 DRV8870TH, U4 DRV8870TH, U5 AS5600, U6 LDO-HT71XX, X1 04-JST-B4B-XH-A, X2 PIN_6X1, X5 PIN_5X1HD

Commit message: small fixes
Parts:
- moved TP1 1.00 mm to (9.10, 0.95)
- moved TP2 1.00 mm to (10.4, 0.95)
Connections:
- net +3V3: now also U2.3, U3.3, U4.3
- net N$3: no longer U3.8
- net N$4: no longer U2.8
- net N$5: no longer U2.3
- net N$6: no longer U3.3
- net N$7: no longer U4.8
- net N$9: no longer U4.3
Routing:
- net +3V3: track 74.2 -> 81.0 mm
- net N$4: track 15.3 -> 11.1 mm, vias 2 -> 1
- net N$3: track 21.4 -> 17.2 mm, vias 2 -> 1
- net N$7: track 23.8 -> 20.8 mm, vias 2 -> 1
- net N$6: track 12.2 -> 9.47 mm
- net N$5: track 15.5 -> 13.2 mm
- net GND: track 42.2 -> 44.0 mm
- net D4: track 20.5 -> 19.5 mm
- net D5: track 17.0 -> 16.2 mm
- net N$9: track 22.4 -> 22.7 mm, vias 0 -> 2
