File: pcb/pcb-bldc-servo-2/pcb-bldc-servo-2.brd (EAGLE design)
At the start: 36.5 x 29 mm, 38 parts, among them J1 03-JST-B3B-XH-A, U1 STM32G030F6P6, U2 DRV8870TH, U3 DRV8870TH, U4 DRV8870TH, U5 AS5600, U6 LDO-HT71XX, X1 04-JST-B4B-XH-A, X2 PIN_6X1, X5 PIN_5X1HD

Commit message: pcb v3 as ordered - moved to pcb folder
Connections:
- net +3V3: now also U5.5
- net GND: no longer U5.5
Routing:
- net +3V3: track 81.0 -> 84.6 mm, vias 3 -> 4
- net GND: track 44.0 -> 41.4 mm, vias 80 -> 79
- net N$25: track 20.5 -> 21.3 mm
Changed lines of the file:
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@@
 <layer number="23" name="tOrigins" color="15" fill="1" visible="yes" active="yes"/>
 <layer number="24" name="bOrigins" color="15" fill="1" visible="yes" active="yes"/>
-<layer number="25" name="tNames" color="7" fill="1" visible="yes" active="yes"/>
-<layer number="26" name="bNames" color="7" fill="1" visible="yes" active="yes"/>
-<layer number="27" name="tValues" color="7" fill="1" visible="yes" active="yes"/>
-<layer number="28" name="bValues" color="7" fill="1" visible="yes" active="yes"/>
+<layer number="25" name="tNames" color="7" fill="1" visible="no" active="yes"/>
+<layer number="26" name="bNames" color="7" fill="1" visible="no" active="yes"/>
+<layer number="27" name="tValues" color="7" fill="1" visible="no" active="yes"/>
+<layer number="28" name="bValues" color="7" fill="1" visible="no" active="yes"/>
 <layer number="29" name="tStop" color="7" fill="3" visible="yes" active="yes"/>
 <layer number="30" name="bStop" color="7" fill="6" visible="yes" active="yes"/>
@@
 <element name="J1" library="bt_con-jst-xh" package="B3B-XH" package3d_urn="urn:adsk.eagle:package:27914046/3" value="03-JST-B3B-XH-A" x="10.54" y="26.65" smashed="yes" rot="R180">
 <attribute name="NAME" x="13.08" y="22.59" size="1.27" layer="21" rot="R180"/>
-<attribute name="VALUE" x="13.08" y="30.46" size="1.27" layer="21" rot="R180"/>
 </element>
 <element name="U5" library="ftobler" package="SOIC-8" package3d_urn="urn:adsk.eagle:package:37121609/2" value="AS5600" x="24.5" y="14.5" smashed="yes" rot="MR0">
@@
 <element name="X1" library="bt_con-jst-xh" package="B4B-XH" package3d_urn="urn:adsk.eagle:package:27914051/3" value="04-JST-B4B-XH-A" x="34.1" y="10.55" smashed="yes" rot="R90">
 <attribute name="NAME" x="30.29" y="6.74" size="1.27" layer="21" rot="R90"/>
-<attribute name="VALUE" x="37.91" y="6.74" size="1.27" layer="21" rot="R90"/>
 </element>
 <element name="U$2" library="bt_con-jst-xh" package="B2B-XH" package3d_urn="urn:adsk.eagle:package:27914040/3" value="02-JST-B3B-XH-A" x="34.1" y="21" smashed="yes" rot="R90">
 <attribute name="NAME" x="30.29" y="17.19" size="1.27" layer="21" rot="R90"/>
-<attribute name="VALUE" x="37.91" y="17.19" size="1.27" layer="21" rot="R90"/>
 </element>
 <element name="C6" library="resistor" library_urn="urn:adsk.eagle:library:348" package="153CLV-1010" package3d_urn="urn:adsk.eagle:package:23413/2" value="470u" x="24.7" y="18.8" smashed="yes" rot="R270">
@@
 <contactref element="C14" pad="2"/>
 <contactref element="U5" pad="8"/>
-<contactref element="U5" pad="5"/>
 <contactref element="C15" pad="2"/>
 <contactref element="U6" pad="1"/>
@@
 <wire x1="20.35" y1="11.65" x2="20.35" y2="11.1" width="0.5" layer="1"/>
 <via x="20.35" y="11.65" extent="1-16" drill="0.3" diameter="0.45"/>
-<wire x1="22.595" y1="17.1162" x2="22.6" y2="17.1212" width="0.3" layer="16"/>
-<wire x1="22.6" y1="19.75" x2="22.6" y2="17.1212" width="0.2" layer="16"/>
-<via x="22.6" y="19.75" extent="1-16" drill="0.3" diameter="0.45"/>
 <wire x1="26.5" y1="17.7" x2="27.2" y2="17.7" width="0.3" layer="16"/>
 <wire x1="26.405" y1="17.1162" x2="26.405" y2="17.605" width="0.3" layer="16"/>
@@
 <wire x1="19.045" y1="15.045" x2="19.045" y2="14.155" width="0.3" layer="1"/>
 <wire x1="18.945" y1="20.655" x2="19.8" y2="19.8" width="0.3" layer="1"/>
-<wire x1="19.8" y1="19.8" x2="19.8" y2="15.8" width="0.3" layer="1"/>
+<wire x1="19.8" y1="19.8" x2="19.8" y2="18.05" width="0.3" layer="1"/>
+<wire x1="19.8" y1="18.05" x2="19.8" y2="15.8" width="0.3" layer="1"/>
 <wire x1="19.8" y1="15.8" x2="19.045" y2="15.045" width="0.3" layer="1"/>
 <via x="19.15" y="9.65" extent="1-16" drill="0.3" diameter="0.45"/>
@@
 <wire x1="9.7" y1="1.9" x2="10.81" y2="1.9" width="0.2" layer="1"/>
 <wire x1="10.81" y1="1.9" x2="10.905" y2="1.995" width="0.2" layer="1"/>
+<contactref element="U5" pad="5"/>
+<wire x1="19.8" y1="18.05" x2="19.85" y2="18.1" width="0.2" layer="1"/>
+<wire x1="19.85" y1="18.1" x2="21.3" y2="18.1" width="0.2" layer="1"/>
+<via x="21.3" y="18.1" extent="1-16" drill="0.3" diameter="0.45"/>
+<wire x1="22.595" y1="17.1162" x2="22.45" y2="17.2612" width="0.2" layer="16"/>
+<wire x1="22.45" y1="17.2612" x2="22.45" y2="18" width="0.2" layer="16"/>
+<wire x1="22.45" y1="18" x2="22.35" y2="18.1" width="0.2" layer="16"/>
+<wire x1="22.35" y1="18.1" x2="21.3" y2="18.1" width="0.2" layer="16"/>
 </signal>
 <signal name="N$3">
@@
 <via x="20.0315875" y="22.7184125" extent="1-16" drill="0.3" diameter="0.45"/>
 <wire x1="20.0315875" y1="22.7184125" x2="20.95" y2="21.8" width="0.2" layer="16"/>
-<wire x1="20.95" y1="21.8" x2="20.95" y2="15.1" width="0.2" layer="16"/>
 <wire x1="20.95" y1="15.1" x2="21.299325" y2="14.750675" width="0.2" layer="16"/>
 <wire x1="21.299325" y1="14.750675" x2="21.550675" y2="14.750675" width="0.2" layer="16"/>
@@
 <wire x1="24.575" y1="10.913175" x2="21.550675" y2="13.9375" width="0.2" layer="15"/>
 <wire x1="24.575" y1="9.525" x2="24.575" y2="10.913175" width="0.2" layer="15"/>
+<wire x1="20.95" y1="21.8" x2="20.95" y2="18.563175" width="0.2" layer="16"/>
+<wire x1="20.95" y1="18.563175" x2="20.725" y2="18.338175" width="0.2" layer="16"/>
+<wire x1="20.725" y1="18.338175" x2="20.725" y2="17.861825" width="0.2" layer="16"/>
+<wire x1="20.725" y1="17.861825" x2="20.95" y2="17.636825" width="0.2" layer="16"/>
+<wire x1="20.95" y1="17.636825" x2="20.95" y2="15.1" width="0.2" layer="16"/>
 </signal>
 <signal name="N$24">
@@
 <wire x1="21.929" y1="13.021" x2="21.65" y2="13.3" width="0.2" layer="1"/>
 <wire x1="21.65" y1="13.3" x2="21.65" y2="13.838175" width="0.2" layer="1"/>
-<wire x1="20.45" y1="15.038175" x2="21.65" y2="13.838175" width="0.2" layer="1"/>
+<wire x1="20.975675" y1="14.5125" x2="21.65" y2="13.838175" width="0.2" layer="1"/>
 <wire x1="18.6" y1="22.3" x2="20.45" y2="20.45" width="0.2" layer="1"/>
-<wire x1="20.45" y1="20.45" x2="20.45" y2="15.038175" width="0.2" layer="1"/>
+<wire x1="20.45" y1="20.45" x2="20.45" y2="19.763175" width="0.2" layer="1"/>
 <wire x1="17.95" y1="22.3" x2="18.9065875" y2="23.2565875" width="0.2" layer="1"/>
 <wire x1="18.9065875" y1="23.2565875" x2="19.1565875" y2="23.2565875" width="0.2" layer="1"/>
@@
 <wire x1="19.4934125" y1="23.5934125" x2="19.4934125" y2="23.7184125" width="0.2" layer="1"/>
 <wire x1="19.4934125" y1="23.7184125" x2="23.175" y2="27.4" width="0.2" layer="1"/>
+<wire x1="20.45" y1="19.763175" x2="21.875" y2="18.338175" width="0.2" layer="1"/>
+<wire x1="20.975675" y1="15.925675" x2="20.975675" y2="14.5125" width="0.2" layer="1"/>
+<wire x1="21.875" y1="18.338175" x2="21.875" y2="16.825" width="0.2" layer="1"/>
+<wire x1="21.875" y1="16.825" x2="20.975675" y2="15.925675" width="0.2" layer="1"/>
 </signal>
 <signal name="NRST">
