File: pcb/pcb-bldc-servo-3/pcb-bldc-servo-3.brd (EAGLE design)
At the start: 36.5 x 29 mm, 45 parts, among them J1 03-JST-B3B-XH-A, U1 STM32G030F6P6, U2 CSD97395Q4M, U3 CSD97395Q4M, U4 CSD97395Q4M, U5 AS5600, U6 LDO-HT71XX, X1 04-JST-B4B-XH-A, X2 PIN_6X1, X5 PIN_5X1HD

Commit message: pcb v3 as ordered - moved to pcb folder
Parts:
- added D4: LED-0805, ftobler:0805-DOT
- added R6: 10k, passives:0603-RES
- added U$3: LOGO-TOBENG-4MM-FINISH, ftobler:TOBENG-4MM-FINISH
- moved TP4 3.86 mm to (19.9, 4.45)
Connections:
- new net N$13: D4.2, R6.2
- net +3V3: now also U5.5
- net D5: now also D4.1
- net GND: now also R6.1; no longer U5.5
Routing:
- net +3V3: track 86.5 -> 91.0 mm, vias 5 -> 6
- net D5: track 13.6 -> 16.2 mm, vias 2 -> 3
- net N$9: track 12.2 -> 13.9 mm
- net GND: track 30.9 -> 29.4 mm, vias 67 -> 66
- net N$13: track 0.00 -> 1.25 mm
- net D6: track 7.55 -> 8.42 mm
- net N$25: track 20.5 -> 21.2 mm
- net MAG_SCL: track 18.4 -> 19.0 mm
Other:
- board text added: "BOTTOM COPPER"
- board text added: "BOTTOM MASK"
- board text added: "BOTTOM SILK"
- board text added: "DIMENSION"
- board text added: "JLCJLCJLCJLCJLC"
- board text added: "MILLING"
- board text added: "TOP COPPER"
- board text added: "TOP MASK"
- board text added: "TOP SILK"
- board text removed: "JLCJLCJLCJLC"
