File: pcb/pcb-bldc-servo-3/pcb-bldc-servo-3.sch (EAGLE design)
At the start: 45 parts, among them J1 03-JST-B3B-XH-A, U1 STM32G030F6P6, U2 CSD97395Q4M, U3 CSD97395Q4M, U4 CSD97395Q4M, U5 AS5600, U6 LDO-HT71XX, X1 04-JST-B4B-XH-A, X2 PIN_6X1, X5 PIN_5X1HD

Commit message: pcb v3 as ordered - moved to pcb folder
Parts:
- added D4: LED-0805, ftobler:LED-0805
- added R6: 10k, passives:RESISTOR0603_RES
- added U$3: LOGO-TOBENG-4MM-FINISH, ftobler:LOGO-TOBENG-4MM-FINISH
Connections:
- new net N$13: D4.2, R6.2
- net +3V3: now also U5.PGO
- net D5: now also D4.1
- net GND: now also R6.1; no longer U5.PGO
Other:
- note added: "General Purpose I/O"
- note added: "Motor"
- note added: "Power Input (6-24V nominal)"
- note added: "ST-Link Programming"
- note removed: "DRV8870 (chinese clone delivers 3.5A continious. But since it is a Brushed DC motor driver, it has some logic that prevents using both outputs in parallel."
- note removed: "Programming"
