File: pcb/pcb-bldc-servo-4/pcb-bldc-servo-4.sch (EAGLE design)
At the start: 51 parts, among them J1 03-JST-B3B-XH-A, U1 STM32G030F6P6, U2 CSD97395Q4M, U3 CSD97395Q4M, U4 CSD97395Q4M, U5 AS5600, U6 LDO-HT71XX, U7 LDO-23, X1 04-JST-B4B-XH-A, X2 PIN_6X1, X5 PIN_5X1HD

Commit message: pcb release v4
Parts:
- U6: value LDO-HT71XX -> HT7150
- U7: value LDO-23 -> HX7133
Changed lines of the file:
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@@
 <part name="C15" library="passives" deviceset="CAPACITOR" device="0603_CAP" package3d_urn="urn:adsk.eagle:package:36813215/3" value="10n"/>
 <part name="GND20" library="supply1" library_urn="urn:adsk.eagle:library:371" deviceset="GND" device=""/>
-<part name="U6" library="ftobler" deviceset="LDO" device="-HT71XX" package3d_urn="urn:adsk.eagle:package:36804013/2"/>
+<part name="U6" library="ftobler" deviceset="LDO" device="-HT71XX" package3d_urn="urn:adsk.eagle:package:36804013/2" value="HT7150"/>
 <part name="C3" library="passives" deviceset="CAPACITOR" device="0603_CAP" package3d_urn="urn:adsk.eagle:package:36813215/3" value="100n"/>
 <part name="C4" library="passives" deviceset="CAPACITOR" device="0603_CAP" package3d_urn="urn:adsk.eagle:package:36813215/3" value="100n"/>
@@
 <part name="R6" library="passives" deviceset="RESISTOR" device="0603_RES" package3d_urn="urn:adsk.eagle:package:36812383/4" value="10k"/>
 <part name="GND30" library="supply1" library_urn="urn:adsk.eagle:library:371" deviceset="GND" device=""/>
-<part name="U7" library="ftobler" deviceset="LDO" device="-23" package3d_urn="urn:adsk.eagle:package:36806100/2" value="LDO-23"/>
+<part name="U7" library="ftobler" deviceset="LDO" device="-23" package3d_urn="urn:adsk.eagle:package:36806100/2" value="HX7133"/>
 <part name="C21" library="passives" deviceset="CAPACITOR" device="0603_CAP" package3d_urn="urn:adsk.eagle:package:36813215/3" value="100n"/>
 <part name="C22" library="passives" deviceset="CAPACITOR" device="0603_CAP" package3d_urn="urn:adsk.eagle:package:36813215/3" value="100n"/>
